Commit message: added mymobi_nav directory for navigations related files

File: mymobi_design/urdf/MYMOBI.urdf (robot description, URDF)
Before this commit: robot MYMOBI, 5 links, 4 joints
Links:
- link b_castor: geometry collision mesh filename=package://mymobi_design/meshes/b_castor.STL; visual mesh filename=package://mymobi_design/meshes/b_castor.STL
- link base_link: geometry collision mesh filename=package://mymobi_design/meshes/base_link.STL; visual mesh filename=package://mymobi_design/meshes/base_link.STL
- link f_castor: geometry collision mesh filename=package://mymobi_design/meshes/f_castor.STL; visual mesh filename=package://mymobi_design/meshes/f_castor.STL
- link l_wheel: geometry collision mesh filename=package://mymobi_design/meshes/l_wheel.STL; visual mesh filename=package://mymobi_design/meshes/l_wheel.STL
- link r_wheel: geometry collision mesh filename=package://mymobi_design/meshes/r_wheel.STL; visual mesh filename=package://mymobi_design/meshes/r_wheel.STL
