Commit message: move base node configured to mymobi

File: mymobi_design/urdf/mymobi.xacro (robot description, xacro)
@@ -308,5 +308,5 @@
   </link>
   <joint name="hokuyo_joint" type="fixed">
-    <origin xyz="${base_radius - hokuyo_size/2} 0 ${base_height+hokuyo_size/4}" rpy="0 0 0" />
+    <origin xyz="0 0.05 ${0.1+hokuyo_size/4}" rpy="0 0 1.5" />
     <parent link="base_link"/>
     <child link="laser_link" />
@@ -324,11 +324,11 @@
             <samples>720</samples>
             <resolution>1</resolution>
-            <min_angle>-1.570796</min_angle>
-            <max_angle>1.570796</max_angle>
+            <min_angle>-1</min_angle> <!--"-1.570796"-->
+            <max_angle>1</max_angle>  <!--"1.570796"-->
           </horizontal>
         </scan>
         <range>
           <min>0.10</min>
-          <max>10.0</max>
+          <max>3.0</max>
           <resolution>0.001</resolution>
         </range>
